File: Eagle/s3-pilot2.brd (EAGLE design)
At the start: 57.1 x 53.6 mm, 18 parts, among them M2_1 ENA

Commit message: OSPARK order 3/29/15
Parts:
- moved R4 30.5 mm to (10.2, 31.8), turned to 90 degrees
- moved R1 16.9 mm to (40.6, 31.8), turned to 90 degrees
- turned ENABLE to 90 degrees
- turned HEARTBEAT to 90 degrees
- turned POWER to 90 degrees
Routing:
- net VDD: track 0.00 -> 123.5 mm, vias 0 -> 1
- net SDA: track 0.00 -> 98.4 mm
- net SCL: track 0.00 -> 90.9 mm
- net M1_A: track 0.00 -> 73.6 mm
- net PWM_X: track 0.00 -> 56.1 mm
- net M1_B: track 0.00 -> 51.3 mm
- net IMU_INT: track 0.00 -> 50.0 mm
- net RESET: track 0.00 -> 49.0 mm
- net M2_A: track 0.00 -> 46.2 mm
- net M1_PWM: track 0.00 -> 37.2 mm
- net M1_DIR: track 0.00 -> 35.7 mm
- net M2_FB: track 0.00 -> 35.2 mm
- net M1_FB: track 0.00 -> 35.1 mm
- net ESC_EN: track 0.00 -> 35.1 mm
- net M2_DIR: track 0.00 -> 35.0 mm
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- added copper zone on layer 1, net GND
- added copper zone on layer 16, net GND
Other:
- board size 57.1 x 53.6 mm -> 57.1 x 53.3 mm
