File: s3-pilot2.brd (EAGLE design)
At the start: 57.1 x 53.3 mm, 18 parts, among them M2_1 ENA

Commit message: update bumper switch
Parts:
- removed R1: 1k, SparkFun-Passives:1206
Connections:
- removed net N$3: JP5.2, R1.2
- net GND: now also JP5.2
- net VDD: no longer R1.1
Routing:
- net N$3: track 18.8 -> 0.00 mm
Changed lines of the file:
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@@
 <attribute name="VALUE" x="17.018" y="30.734" size="0.6096" layer="27" rot="R90"/>
-</element>
-<element name="R1" library="SparkFun-Passives" package="1206" value="1k" x="40.64" y="31.75" smashed="yes" rot="R90">
-<attribute name="NAME" x="39.497" y="29.21" size="1.016" layer="25" rot="R90"/>
-<attribute name="VALUE" x="39.624" y="32.893" size="1.016" layer="27" rot="R90"/>
 </element>
 <element name="R4" library="SparkFun-Passives" package="1206" value="1k" x="10.16" y="31.75" smashed="yes" rot="R90">
@@
 <wire x1="34.2392" y1="7.62" x2="34.162984375" y2="7.62" width="0.508" layer="16"/>
 <wire x1="31.9024" y1="7.5184" x2="31.75" y2="7.62" width="0.508" layer="16"/>
+<contactref element="JP5" pad="2"/>
 </signal>
 <signal name="VDD" class="1">
@@
 <contactref element="U$1" pad="VDD"/>
 <contactref element="U$3" pad="VDD"/>
-<contactref element="R1" pad="1"/>
 <contactref element="JP2" pad="2"/>
 <contactref element="JP4" pad="1"/>
@@
 <wire x1="35.56" y1="25.4" x2="39.2684" y2="29.1084" width="0.508" layer="1"/>
 <wire x1="39.2684" y1="29.1084" x2="40.4368" y2="30.2768" width="0.508" layer="1"/>
-<wire x1="40.64" y1="30.2768" x2="40.64" y2="30.35" width="0.508" layer="1"/>
 <wire x1="35.56" y1="25.4" x2="33.02" y2="25.4" width="0.508" layer="1"/>
 <wire x1="50.5968" y1="17.78" x2="50.8" y2="17.78" width="0.508" layer="16"/>
@@
 <wire x1="46.9392" y1="7.62" x2="46.99" y2="7.62" width="0.2032" layer="16"/>
 </signal>
-<signal name="N$3">
-<contactref element="R1" pad="2"/>
-<contactref element="JP5" pad="2"/>
-<wire x1="40.64" y1="35.3568" x2="40.64" y2="33.15" width="0.2032" layer="1"/>
-<wire x1="45.0088" y1="39.7256" x2="40.64" y2="35.3568" width="0.2032" layer="1"/>
-<wire x1="45.0088" y1="42.3672" x2="45.0088" y2="39.7256" width="0.2032" layer="1"/>
-<wire x1="49.5808" y1="46.9392" x2="45.0088" y2="42.3672" width="0.2032" layer="1"/>
-<wire x1="50.8" y1="46.9392" x2="49.5808" y2="46.9392" width="0.2032" layer="1"/>
-<wire x1="50.8" y1="46.9392" x2="50.8" y2="46.99" width="0.2032" layer="1"/>
-</signal>
 <signal name="3.3">

Commit message: started new version.
Connections:
- net BUMPER: now also JP5.2; no longer JP5.1
- net GND: now also JP5.1; no longer JP5.2
Routing:
- net BUMPER: track 9.01 -> 30.0 mm
- net GND: track 0.62 -> 1.89 mm
Changed lines of the file:
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@@
 <?xml version="1.0" encoding="utf-8"?>
 <!DOCTYPE eagle SYSTEM "eagle.dtd">
-<eagle version="7.2.0">
+<eagle version="7.3.0">
 <drawing>
 <settings>
@@
 <vertex x="57.15" y="58.42"/>
 </polygon>
-<wire x1="34.2392" y1="7.62" x2="34.29" y2="7.62" width="0.508" layer="1"/>
-<wire x1="34.2392" y1="7.62" x2="34.162984375" y2="7.62" width="0.508" layer="1"/>
+<wire x1="34.29" y1="7.62" x2="34.162984375" y2="7.62" width="0.508" layer="1"/>
 <wire x1="31.9024" y1="7.5184" x2="31.75" y2="7.62" width="0.508" layer="1"/>
-<wire x1="34.2392" y1="7.62" x2="34.29" y2="7.62" width="0.508" layer="16"/>
-<wire x1="34.2392" y1="7.62" x2="34.162984375" y2="7.62" width="0.508" layer="16"/>
+<wire x1="34.29" y1="7.62" x2="34.162984375" y2="7.62" width="0.508" layer="16"/>
 <wire x1="31.9024" y1="7.5184" x2="31.75" y2="7.62" width="0.508" layer="16"/>
-<contactref element="JP5" pad="2"/>
+<contactref element="JP5" pad="1"/>
+<wire x1="5.08" y1="47.625" x2="5.08" y2="48.26" width="0.508" layer="16"/>
+<wire x1="5.08" y1="48.895" x2="5.08" y2="48.26" width="0.508" layer="16"/>
 </signal>
 <signal name="VDD" class="1">
@@
 <signal name="BUMPER">
 <contactref element="GND" pad="D4"/>
-<contactref element="JP5" pad="1"/>
 <wire x1="44.5008" y1="55.88" x2="50.8" y2="49.5808" width="0.2032" layer="1"/>
-<wire x1="50.8" y1="49.5808" x2="50.8" y2="49.53" width="0.2032" layer="1"/>
 <wire x1="44.5008" y1="55.88" x2="44.45" y2="55.88" width="0.2032" layer="1"/>
+<contactref element="JP5" pad="2"/>
+<wire x1="53.34" y1="46.99" x2="50.8" y2="46.99" width="0.2032" layer="1"/>
+<wire x1="53.34" y1="52.705" x2="53.34" y2="46.99" width="0.2032" layer="1"/>
+<wire x1="50.8" y1="55.245" x2="53.34" y2="52.705" width="0.2032" layer="1"/>
+<wire x1="50.8" y1="56.515" x2="50.8" y2="55.245" width="0.2032" layer="1"/>
+<wire x1="50.165" y1="57.15" x2="50.8" y2="56.515" width="0.2032" layer="1"/>
+<wire x1="44.45" y1="57.15" x2="50.165" y2="57.15" width="0.2032" layer="1"/>
+<wire x1="44.45" y1="55.88" x2="44.45" y2="57.15" width="0.2032" layer="1"/>
 </signal>
 <signal name="M1_PWM">
