File: s3-pilot2.sch (EAGLE design)
At the start: 18 parts, among them M2_1 ENA

Commit message: update bumper switch
Parts:
- removed R1: 1k, SparkFun-Passives:RESISTOR1206
Connections:
- removed net N$3: JP5.2, R1.2
- net GND: now also JP5.2
- net VDD: no longer R1.1
Other:
- note added: "4/18/2015 switch bumper to gnd"
- note added: "revisions:"
Changed lines of the file:
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@@
 <part name="GND5" library="SparkFun-Aesthetics" deviceset="GND" device=""/>
 <part name="JP2" library="pinhead" deviceset="PINHD-1X3" device="/90" value="PWMX"/>
-<part name="R1" library="SparkFun-Passives" deviceset="RESISTOR" device="1206" value="1k"/>
 <part name="GND9" library="SparkFun-Aesthetics" deviceset="GND" device=""/>
-<part name="SUPPLY8" library="SparkFun-Aesthetics" deviceset="VDD" device=""/>
 <part name="SUPPLY9" library="SparkFun-Aesthetics" deviceset="VDD" device=""/>
 <part name="RESET" library="SparkFun-Electromechanical" deviceset="SWITCH-MOMENTARY-2" device="SMD-4" value="RESET"/>
@@
 <part name="GND4" library="SparkFun-Aesthetics" deviceset="GND" device=""/>
 <part name="JP1" library="pinhead" deviceset="PINHD-1X2" device="" value="Reset"/>
+<part name="GND6" library="SparkFun-Aesthetics" deviceset="GND" device=""/>
 </parts>
 <sheets>
 <sheet>
 <plain>
+<text x="48.26" y="25.4" size="1.778" layer="91">revisions:</text>
+<text x="50.8" y="20.32" size="1.778" layer="91">4/18/2015 switch bumper to gnd</text>
 </plain>
 <instances>
@@
 <instance part="GND5" gate="1" x="177.8" y="50.8" rot="R90"/>
 <instance part="JP2" gate="A" x="162.56" y="160.02" rot="R90"/>
-<instance part="R1" gate="G$1" x="134.62" y="142.24" rot="R90"/>
 <instance part="GND9" gate="1" x="160.02" y="144.78"/>
-<instance part="SUPPLY8" gate="VDD" x="134.62" y="137.16" rot="R180"/>
 <instance part="SUPPLY9" gate="VDD" x="162.56" y="134.62" rot="R180"/>
 <instance part="RESET" gate="G$1" x="220.98" y="132.08" rot="R90"/>
@@
 <instance part="GND4" gate="1" x="50.8" y="60.96" rot="R270"/>
 <instance part="JP1" gate="G$1" x="236.22" y="157.48" rot="R90"/>
+<instance part="GND6" gate="1" x="134.62" y="142.24"/>
 </instances>
 <busses>
@@
 <wire x1="53.34" y1="60.96" x2="53.34" y2="68.58" width="0.1524" layer="91"/>
 </segment>
+<segment>
+<wire x1="134.62" y1="157.48" x2="134.62" y2="144.78" width="0.1524" layer="91"/>
+<pinref part="JP5" gate="G$1" pin="2"/>
+<pinref part="GND6" gate="1" pin="GND"/>
+</segment>
 </net>
 <net name="VDD" class="1">
@@
 <wire x1="73.66" y1="63.5" x2="73.66" y2="66.04" width="0.1524" layer="91"/>
 <junction x="73.66" y="66.04"/>
-</segment>
-<segment>
-<pinref part="R1" gate="G$1" pin="1"/>
-<pinref part="SUPPLY8" gate="VDD" pin="VDD"/>
 </segment>
 <segment>
@@
 </segment>
 </net>
-<net name="N$3" class="0">
-<segment>
-<wire x1="134.62" y1="157.48" x2="134.62" y2="147.32" width="0.1524" layer="91"/>
-<pinref part="R1" gate="G$1" pin="2"/>
-<pinref part="JP5" gate="G$1" pin="2"/>
-</segment>
-</net>

Commit message: started new version.
Connections:
- net BUMPER: now also JP5.2; no longer JP5.1
- net GND: now also JP5.1; no longer JP5.2
Other:
- moved on the sheet: JP1, JP3, JP4, JP5, M2_1
Changed lines of the file:
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@@
 <?xml version="1.0" encoding="utf-8"?>
 <!DOCTYPE eagle SYSTEM "eagle.dtd">
-<eagle version="7.2.0">
+<eagle version="7.3.0">
 <drawing>
 <settings>
@@
 <part name="GND4" library="SparkFun-Aesthetics" deviceset="GND" device=""/>
 <part name="JP1" library="pinhead" deviceset="PINHD-1X2" device="" value="Reset"/>
-<part name="GND6" library="SparkFun-Aesthetics" deviceset="GND" device=""/>
 </parts>
 <sheets>
@@
 <instance part="R4" gate="G$1" x="195.58" y="124.46" rot="R90"/>
 <instance part="R8" gate="G$1" x="208.28" y="124.46" rot="R90"/>
-<instance part="M2_1" gate="G$1" x="139.7" y="114.3" rot="R180"/>
+<instance part="M2_1" gate="G$1" x="127" y="124.46" rot="R180"/>
 <instance part="GND1" gate="1" x="220.98" y="111.76"/>
 <instance part="SUPPLY1" gate="VDD" x="243.84" y="30.48" rot="R180"/>
@@
 <instance part="SUPPLY9" gate="VDD" x="162.56" y="134.62" rot="R180"/>
 <instance part="RESET" gate="G$1" x="220.98" y="132.08" rot="R90"/>
-<instance part="JP3" gate="A" x="142.24" y="91.44" rot="R180"/>
-<instance part="JP4" gate="A" x="142.24" y="73.66" rot="R180"/>
-<instance part="JP5" gate="G$1" x="134.62" y="160.02" rot="R90"/>
+<instance part="JP3" gate="A" x="127" y="104.14" rot="R180"/>
+<instance part="JP4" gate="A" x="127" y="81.28" rot="R180"/>
+<instance part="JP5" gate="G$1" x="248.92" y="157.48" rot="R90"/>
 <instance part="GND3" gate="1" x="50.8" y="109.22" rot="R270"/>
 <instance part="GND4" gate="1" x="50.8" y="60.96" rot="R270"/>
-<instance part="JP1" gate="G$1" x="236.22" y="157.48" rot="R90"/>
-<instance part="GND6" gate="1" x="134.62" y="142.24"/>
+<instance part="JP1" gate="G$1" x="233.68" y="157.48" rot="R90"/>
 </instances>
 <busses>
@@
 </segment>
 <segment>
-<wire x1="144.78" y1="71.12" x2="154.94" y2="71.12" width="0.1524" layer="91"/>
-<label x="160.02" y="71.12" size="1.778" layer="95" rot="R180"/>
+<wire x1="129.54" y1="78.74" x2="139.7" y2="78.74" width="0.1524" layer="91"/>
+<label x="137.16" y="78.74" size="1.778" layer="95"/>
 <pinref part="JP4" gate="A" pin="2"/>
 </segment>
 <segment>
-<wire x1="144.78" y1="88.9" x2="154.94" y2="88.9" width="0.1524" layer="91"/>
-<label x="160.02" y="88.9" size="1.778" layer="95" rot="R180"/>
+<wire x1="129.54" y1="101.6" x2="139.7" y2="101.6" width="0.1524" layer="91"/>
+<label x="137.16" y="101.6" size="1.778" layer="95"/>
 <pinref part="JP3" gate="A" pin="2"/>
 </segment>
@@
 <pinref part="RESET" gate="G$1" pin="1"/>
 <pinref part="JP1" gate="G$1" pin="1"/>
-<wire x1="220.98" y1="116.84" x2="233.68" y2="116.84" width="0.1524" layer="91"/>
-<wire x1="233.68" y1="116.84" x2="233.68" y2="154.94" width="0.1524" layer="91"/>
+<wire x1="220.98" y1="116.84" x2="231.14" y2="116.84" width="0.1524" layer="91"/>
+<wire x1="231.14" y1="116.84" x2="231.14" y2="154.94" width="0.1524" layer="91"/>
+<pinref part="JP5" gate="G$1" pin="1"/>
+<wire x1="246.38" y1="154.94" x2="246.38" y2="116.84" width="0.1524" layer="91"/>
+<wire x1="246.38" y1="116.84" x2="231.14" y2="116.84" width="0.1524" layer="91"/>
+<junction x="231.14" y="116.84"/>
 </segment>
 <segment>
@@
 <wire x1="53.34" y1="60.96" x2="53.34" y2="68.58" width="0.1524" layer="91"/>
 </segment>
-<segment>
-<wire x1="134.62" y1="157.48" x2="134.62" y2="144.78" width="0.1524" layer="91"/>
-<pinref part="JP5" gate="G$1" pin="2"/>
-<pinref part="GND6" gate="1" pin="GND"/>
-</segment>
 </net>
 <net name="VDD" class="1">
@@
 </segment>
 <segment>
-<wire x1="144.78" y1="68.58" x2="154.94" y2="68.58" width="0.1524" layer="91"/>
-<label x="160.02" y="68.58" size="1.778" layer="95" rot="R180"/>
+<wire x1="129.54" y1="76.2" x2="139.7" y2="76.2" width="0.1524" layer="91"/>
+<label x="137.16" y="76.2" size="1.778" layer="95"/>
 <pinref part="JP4" gate="A" pin="1"/>
 </segment>
 <segment>
-<wire x1="144.78" y1="86.36" x2="154.94" y2="86.36" width="0.1524" layer="91"/>
-<label x="160.02" y="86.36" size="1.778" layer="95" rot="R180"/>
+<wire x1="129.54" y1="99.06" x2="139.7" y2="99.06" width="0.1524" layer="91"/>
+<label x="137.16" y="99.06" size="1.778" layer="95"/>
 <pinref part="JP3" gate="A" pin="1"/>
 </segment>
@@
 <net name="M1_B" class="0">
 <segment>
-<wire x1="144.78" y1="93.98" x2="154.94" y2="93.98" width="0.1524" layer="91"/>
-<label x="160.02" y="93.98" size="1.778" layer="95" rot="R180"/>
+<wire x1="129.54" y1="106.68" x2="139.7" y2="106.68" width="0.1524" layer="91"/>
+<label x="137.16" y="106.68" size="1.778" layer="95"/>
 <pinref part="JP3" gate="A" pin="4"/>
 </segment>
@@
 <net name="M1_A" class="0">
 <segment>
-<wire x1="144.78" y1="91.44" x2="154.94" y2="91.44" width="0.1524" layer="91"/>
-<label x="160.02" y="91.44" size="1.778" layer="95" rot="R180"/>
+<wire x1="129.54" y1="104.14" x2="139.7" y2="104.14" width="0.1524" layer="91"/>
+<label x="137.16" y="104.14" size="1.778" layer="95"/>
 <pinref part="JP3" gate="A" pin="3"/>
 </segment>
@@
 <net name="M2_B" class="0">
 <segment>
-<wire x1="144.78" y1="76.2" x2="154.94" y2="76.2" width="0.1524" layer="91"/>
-<label x="160.02" y="76.2" size="1.778" layer="95" rot="R180"/>
+<wire x1="129.54" y1="83.82" x2="139.7" y2="83.82" width="0.1524" layer="91"/>
+<label x="137.16" y="83.82" size="1.778" layer="95"/>
 <pinref part="JP4" gate="A" pin="4"/>
 </segment>
@@
 <net name="M2_A" class="0">
 <segment>
-<wire x1="144.78" y1="73.66" x2="154.94" y2="73.66" width="0.1524" layer="91"/>
-<label x="160.02" y="73.66" size="1.778" layer="95" rot="R180"/>
+<wire x1="129.54" y1="81.28" x2="139.7" y2="81.28" width="0.1524" layer="91"/>
+<label x="137.16" y="81.28" size="1.778" layer="95"/>
 <pinref part="JP4" gate="A" pin="3"/>
 </segment>
@@
 </segment>
 <segment>
-<wire x1="132.08" y1="157.48" x2="132.08" y2="144.78" width="0.1524" layer="91"/>
-<wire x1="132.08" y1="144.78" x2="127" y2="144.78" width="0.1524" layer="91"/>
-<label x="121.92" y="144.78" size="1.778" layer="95"/>
-<pinref part="JP5" gate="G$1" pin="1"/>
+<wire x1="248.92" y1="154.94" x2="248.92" y2="142.24" width="0.1524" layer="91"/>
+<pinref part="JP5" gate="G$1" pin="2"/>
+<label x="248.92" y="139.7" size="1.778" layer="95" rot="R90"/>
 </segment>
 </net>
@@
 <segment>
 <pinref part="M2_1" gate="G$1" pin="2"/>
-<wire x1="142.24" y1="114.3" x2="152.4" y2="114.3" width="0.1524" layer="91"/>
-<label x="162.56" y="114.3" size="1.778" layer="95" rot="R180"/>
+<wire x1="129.54" y1="124.46" x2="139.7" y2="124.46" width="0.1524" layer="91"/>
+<label x="137.16" y="124.46" size="1.778" layer="95"/>
 </segment>
 </net>
@@
 <segment>
 <pinref part="JP1" gate="G$1" pin="2"/>
-<wire x1="236.22" y1="154.94" x2="236.22" y2="144.78" width="0.1524" layer="91"/>
-<label x="236.22" y="142.24" size="1.778" layer="95" rot="R90"/>
+<wire x1="233.68" y1="154.94" x2="233.68" y2="144.78" width="0.1524" layer="91"/>
+<label x="233.68" y="142.24" size="1.778" layer="95" rot="R90"/>
 </segment>
 </net>
@@
 <segment>
 <pinref part="M2_1" gate="G$1" pin="1"/>
-<wire x1="142.24" y1="111.76" x2="152.4" y2="111.76" width="0.1524" layer="91"/>
-<label x="162.56" y="111.76" size="1.778" layer="95" rot="R180"/>
-</segment>
-<segment>
+<wire x1="129.54" y1="121.92" x2="139.7" y2="121.92" width="0.1524" layer="91"/>
+<label x="137.16" y="121.92" size="1.778" layer="95"/>
+</segment>
+<segment>
