File: s3-pilot3.sch (EAGLE design)
At the start: 88 parts, among them IC3 LM1117, IC4 ATMEGA1284, J1 POWER_JACKOVERPASTE_REDBOARD_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, J2 ICSP, M2_1 ENA, Q1 ZXMP6A13FTA, Q2 2N7002PW, U1 FT231XS, U2 MIC5205, U3 ATMEGA328, X2 JTAG, X3 USB, X5 UART0, Y1 16MHz, Y2 16MHz

Commit message: .
Parts:
- removed AD: (no value), SparkFun:M06SMD-STRAIGHT-COMBO
- removed C1, C2, C8: 0.1uF, SparkFun:CAP0603-CAP
- removed C21: 100n, SparkFun:CAPPTH
- removed ENABLE: RED, SparkFun-LED:LED-RED1206
- removed F2: PTCPTH, SparkFun:PTCPTH
- removed GND: ARDUINO_R3_SHIELD, SparkFun-Boards:ARDUINO_R3_SHIELD
- removed HEARTBEAT: BLUE, SparkFun-LED:LED-BLUE1206
- removed IOL: (no value), SparkFun:M08SMD-COMBO
- removed J1: POWER_JACKOVERPASTE_REDBOARD_0603, Testing:POWER_JACKOVERPASTE_REDBOARD_0603
- removed J2: ICSP, SparkFun-Connectors:AVR_SPI_PRG_6SMT_MALE
- removed M2_1: ENA, pinhead:PINHD-1X2
- removed POWER: GREEN, SparkFun-LED:LED-GREENLARGE
- removed R4, R6, R8: 1k, SparkFun-Passives:RESISTOR1206
- removed S1: RESET, SparkFun:TAC_SWITCHSMD
- removed TP1, TP2, TP3, TP4, TP5, TP6: TP-3x5, SparkFun-Passives:TEST-POINT3X5
- removed U$3: M2, s3-pilot2-lbr:MC33926-SINGLE-BO
- removed U3: ATMEGA328, SparkFun:ATMEGA168
- removed X2: JTAG, SteveMarple:ATMEL-JTAG
- removed X3: USB, SteveMarple:USBPTH
- removed X5: UART0, SparkFun:ARDUINO_SERIAL_PROGRAMPTH
- removed Y1: 16MHz, SparkFun-FreqCtrl:RESONATORSMD
- added 5V_IN, PI_PWR, PI_SW: (no value), pinhead:PINHD-1X2
- added JP11: PWM2, pinhead:PINHD-1X3/90
- added JP12: PWM3, pinhead:PINHD-1X3/90
- added JP13: PWM4, pinhead:PINHD-1X3/90
- added JPX1, JPX8: (no value), pinhead:PINHD-1X12
- added JPX10: (no value), pinhead:PINHD-1X8
- added JTAG: (no value), pinhead:PINHD-2X5
- added LED5: HeartBeat, SparkFun-LED:LED-RED1206
- added U$4: M2, s3-pilot2-lbr:MC33926-SINGLE-BO
- IC3: device Testing:V_REG_LM1117ALT1 -> Testing:V_REG_LM1117SOT223
- JP10: value (none) -> PWM1; device SparkFun-Connectors:M08SMD-COMBO -> pinhead:PINHD-1X3/90
- JP2: value PWMX -> ESC_ENA; device pinhead:PINHD-1X3/90 -> pinhead:PINHD-1X2
- JP6: value M10SMD_COMBO -> M2; device SparkFun-Connectors:M10SMD_COMBO -> pinhead:PINHD-1X12
- JP7: value AUTO RST -> M1; device SparkFun:JUMPER-2PTH -> pinhead:PINHD-1X12
- JP9: value USB/FTDI -> MPU-6050; device SparkFun:JUMPER-3PTH -> pinhead:PINHD-1X8
- LED1: value Blue -> ESC; device SparkFun-LED:LED1206-NS -> SparkFun-LED:LED-RED1206
- LED2: value Green -> Power; device SparkFun-LED:LED1206-NS -> SparkFun-LED:LED1206
- LED3: value Red -> TX; device SparkFun-LED:LED1206-NS -> SparkFun-LED:LED1206
- LED4: value Yellow -> RX; device SparkFun-LED:LED1206-NS -> SparkFun-LED:LED1206
- R3: value 10k -> 1k
- U$1: value M1 -> M2
Connections:
- removed net +5V: F2.2
- removed net +5V_USB: F2.1, JP9.2
- removed net 20(SDA): IC4.PCINT17/SDA_PC1
- removed net 21(SCL): IC4.PCINT16/SCL_PC0
- removed net 23: IC4.PCINT31/OC2A_PD7
- removed net 3.3: GND.3.3V, MPU6050.VCC
- removed net AD0: AD.1, U3.PC0(ADC0)
- removed net AD1: AD.2, U3.PC1(ADC1)
- removed net AD2: AD.3, U3.PC2(ADC2)
- removed net AD3: AD.4, U3.PC3(ADC3)
- removed net AD4/SDA: AD.5, JP6.2, U3.PC4(ADC4/SDA)
- removed net AD5/SCL: AD.6, JP6.1, U3.PC5(ADC5/SCL)
- removed net AUTO_RESET: JP7.1, X5.DTR
- removed net BUMPER: GND.D4, JP5.2
- removed net ESC_EN: ENABLE.A, M2_1.1, U$1.EN, U$3.EN
- removed net IMU_INT: GND.D7, MPU6050.INT
- removed net INSERT: J1.GND, Q1.G, R5.1
- removed net IO2: IOL.3, U3.PD2(INT0)
- removed net IO3: IOL.4, U3.PD3(INT1)
- removed net IO4: IOL.5, U3.PD4(XCK/T0)
- removed net IO5: IOL.6, U3.PD5(T1)
- removed net IO6: IOL.7, U3.PD6(AIN0)
- removed net IO7: IOL.8, U3.PD7(AIN1)
- removed net IO8: JP6.10, U3.PB0(ICP)
- removed net IO9: JP6.9, U3.PB1(OC1A)
- removed net MISO: J2.1, JP6.6, TP4.1, U3.PB4(MISO)
- removed net MOSI: J2.4, JP6.7, TP2.1, U3.PB3(MOSI/OC2)
- removed net PWM_X: GND.*D10, JP2.3
- removed net PWRIN: D1.A, J1.PWR
- removed net RESET: C8.2, GND.RES, J2.5, JP1.2, JP10.6, R3.1, RESET.2, S1.3, S1.4, TP6.1, U3.PC6(/RESET)
- removed net RX-I: IOL.1, R10.1, U3.PD0(RXD)
- removed net SCK: J2.3, JP6.5, R1.1, TP5.1, U3.PB5(SCK)
- removed net SCL: GND.A5, GND.SCL, MPU6050.SCL
- removed net SDA: GND.A4, GND.SDA, MPU6050.SDA
- removed net SS: JP6.8, U3.PB2(SS/OC1B)
- removed net TX-O: IOL.2, R11.1, U3.PD1(TXD)
- removed net USB_D+: X3.D+
- removed net USB_D-: X3.D-
- removed net VCC: C19.1, C20.+, IC4.VCC, L1.2, X2.VTREF
- removed net VDD: GND.5V, JP2.2, JP3.1, JP4.1, POWER.A, U$1.IN2, U$1.VDD, U$3.IN2, U$3.VDD
- new net !BUMPER: JP5.2
- new net ESC_ENA: JP2.1, JP6.3, JP7.3, R3.2
- new net N$14: JPX10.2, MPU6050.AD0
- new net N$17: JPX10.4, MPU6050.XDA
- new net N$18: JPX1.1, U$1.INV
- new net N$19: JPX10.5, MPU6050.SDA
- new net N$20: JPX10.6, MPU6050.SCL
- new net N$22: JPX10.7, MPU6050.GND
- new net N$25: JPX1.2, U$1.SLEW
- new net N$26: IC4.PCINT16/SCL_PC0, JP9.6
- new net N$27: JPX8.4, U$4.FB
- new net N$28: JPX8.5, U$4.!SF
- new net N$29: JPX8.6, U$4.!PWM!_D1
- new net N$30: JPX8.7, U$4.PWM_!D2
- new net N$31: JPX8.8, U$4.IN1
- new net N$32: JPX8.9, U$4.IN2
- new net N$33: JPX8.10, U$4.VDD
- new net N$34: JPX8.11, U$4.GND
- new net N$35: JPX8.12, U$4.VIN
- new net N$36: 5V_IN.2, D1.A
- new net N$37: JPX1.3, U$1.EN
- new net N$38: JPX1.4, U$1.FB
- new net N$39: JPX1.5, U$1.!SF
- new net N$40: PI_PWR.2, PI_SW.1
- new net N$41: JPX1.6, U$1.!PWM!_D1
- new net N$42: JPX1.7, U$1.PWM_!D2
- new net N$43: JPX1.8, U$1.IN1
- new net N$44: JPX1.9, U$1.IN2
- new net N$45: JPX1.10, U$1.VDD
- new net N$46: JPX1.11, U$1.GND
- new net N$47: JPX1.12, U$1.VIN
- new net PWM1: JP10.3
- new net PWM2: JP11.3
- new net PWM3: JP12.3
- new net PWM4: JP13.3
- net !RESET: now also JP1.2, JTAG.6, RESET.2; no longer C21.2, X2.!SRST
- net 0(RX0): now also R10.1; no longer X5.TXO
- net 1(TX0): now also R11.1; no longer X5.RXI
- net 16(TDI): now also JTAG.9; no longer X2.TDI
- net 17(TDO): now also JTAG.3; no longer X2.TDO
- net 18(TMS): now also JTAG.5; no longer X2.TMS
- net 19(TCK): now also JTAG.1; no longer X2.TCK
- net 3.3V: no longer JP10.5
- net 5V: now also C19.1, C20.+, IC4.VCC, JP3.1, JP4.1, JP6.10, JP6.9, JP7.10, JP7.9, JP9.8, JPX10.8, JTAG.4, L1.2, MPU6050.VCC; no longer C2.2, J2.2, JP10.4, JP10.7, R3.2, TP1.1, U3.AVCC, U3.VCC@1, U3.VCC@2
- net A0: now also JP9.1
- net AREF: no longer C1.1, JP6.3, U3.AREF
- net DTR: no longer C8.1
- net ESC_EN_JMP: now also JP2.2; no longer GND.D12, M2_1.2
- net GND: now also JP10.1, JP11.1, JP12.1, JP13.1, JP6.11, JP6.6, JP6.8, JP7.11, JP7.6, JP7.8, JP9.7, JTAG.10, JTAG.2, LED5.C, PI_PWR.1; no longer C1.2, C2.1, GND.GND@0, GND.GND@1, GND.GND@2, J1.GNDBREAK, J2.6, JP10.2, JP10.3, JP2.1, JP6.4, MPU6050.AD0, MPU6050.GND, R4.1, R6.1, R8.1, S1.1, S1.2, TP3.1, U$1.!PWM!_D1, U$1.GND, U$1.IN1, U$3.!PWM!_D1, U$3.GND, U$3.IN1, U3.AGND, U3.GND@1, U3.GND@2, X2.GND@0, X2.GND@1, X3.GND, X5.GND, Y1.2
- net HB: now also R1.2; no longer GND.D13, HEARTBEAT.A
- net M1_A: no longer GND.D2
- net M1_B: no longer GND.D8
- net M1_DIR: now also JP7.1; no longer GND.*D11, U$1.INV
- net M1_FB: now also JP7.5; no longer GND.A2, U$1.FB
- net M1_PWM: now also JP7.7; no longer GND.*D5, U$1.PWM_!D2
- net M2_A: no longer GND.*D3
- net M2_B: no longer GND.*D9
- net M2_DIR: now also JP6.1; no longer GND.A3, U$3.INV
- net M2_FB: now also JP6.5; no longer GND.A1, U$3.FB
- net M2_PWM: now also JP6.7; no longer GND.*D6, U$3.PWM_!D2
- net N$1: now also JPX8.1, U$4.INV; no longer LED1.A, R1.2
- net N$11: now also IC4.PCINT17/SDA_PC1, JP9.5; no longer JP9.1, X5.VCC
- net N$13: now also JPX10.1, MPU6050.INT; no longer C21.1, JP7.2
- net N$16: now also JPX10.3, MPU6050.XCL; no longer JP9.3, X3.VBUS
- net N$21: now also LED5.A, R1.1; no longer POWER.C, R4.2
- net N$23: now also LED1.A, R3.1; no longer ENABLE.C, R8.2
- net N$24: now also 5V_IN.1, Q1.G, R5.1; no longer HEARTBEAT.C, R6.2
- net N$3: now also JPX8.2, U$4.SLEW; no longer U3.PB6(XTAL1/TOSC1), Y1.1
- net N$4: now also JPX8.3, U$4.EN; no longer U3.PB7(XTAL2/TOSC2), Y1.3
- net VIN: now also JP10.2, JP11.2, JP12.2, JP13.2, PI_SW.2; no longer JP10.1
Other:
- note added: "5V in from RC 5A switched regulator. Routed to Pi BUS via switch(or jumper). Also supplies Servos / Pings."
- note added: "Do I need AREF or AVCC?"
- note added: "USB Host for Pi Power"
- note removed: "JTAG header"
- note removed: "notes; use screw term for non usb power in"
- note removed: "todo; merge replace with spark fun arduino swap to 64k chip add 4 servos (1 pin plus power) add 4 ultrasonics (2 pins + power)"
- moved on the sheet: C10, C11, C12, C13, C14, C15, C16, C17, C18, C19, C20, C3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

Commit message: .
Parts:
- removed C11, C16: 22p, SparkFun:CAPPTH
- removed C17, C18, C19: 100n, SparkFun:CAPPTH
- removed C20: 4u7, SparkFun:CAP_POLPTH2
- removed IC4: ATMEGA1284, SteveMarple:ATMEGA644-20PU
- removed JP12: PWM3, pinhead:PINHD-1X3/90
- removed JP13: PWM4, pinhead:PINHD-1X3/90
- removed L1: 10uH, SteveMarple:INDUCTOR0.4"-AXIAL
- removed PI_PWR, PI_SW: (no value), pinhead:PINHD-1X2
- removed Y2: 16MHz, SteveMarple:CRYSTAL-RESONATOR
- added C1, C2: 22p, SparkFun:CAPPTH
- added C21: 4u7, SparkFun:CAP_POLPTH2
- added C8: 100n, SparkFun:CAPPTH
- added IC1: ATMEGA644A, atmel:ATMEGA644A
- added JP14: US2, pinhead:PINHD-1X4/90
- added JP20: SW_1, pinhead:PINHD-1X2
- added JP21: 5V_1, pinhead:PINHD-1X2
- added JP8: MPU-6050, pinhead:PINHD-1X8
- added Y1: 16MHz, SteveMarple:CRYSTAL-RESONATOR
- JP9: value MPU-6050 -> US1; device pinhead:PINHD-1X8 -> pinhead:PINHD-1X4/90
Connections:
- removed net 10: IC4.PCINT12/OC0B/SS_PB4
- removed net 11(MOSI): IC4.PCINT13/MOSI_PB5
- removed net 12(MISO): IC4.PCINT14/MISO_PB6
- removed net 13(SCK): IC4.PCINT15/SCK_PB7
- removed net 14: IC4.PCINT23/TOSC2_PC7
- removed net 15: IC4.PCINT22/TOSC1_PC6
- removed net 16(TDI): IC4.PCINT21/TDI_PC5, JTAG.9
- removed net 17(TDO): IC4.PCINT20/TDO_PC4, JTAG.3
- removed net 18(TMS): IC4.PCINT19/TMS_PC3, JTAG.5
- removed net 19(TCK): IC4.PCINT18/TCK_PC2, JTAG.1
- removed net 2(RX1): IC4.PCINT26/INT0_PD2
- removed net 22: IC4.PCINT28/OC1B_PD4
- removed net 3(TX1): IC4.PCINT27/INT1_PD3
- removed net 4: IC4.PCINT8/XCK0/T0_PB0
- removed net 5: IC4.PCINT9/CLKO/T1_PB1
- removed net 6: IC4.PCINT10/INT2/AIN0_PB2
- removed net 7: IC4.PCINT11/OC0A/AIN1_PB3
- removed net 8: IC4.PCINT30/OC2B/ICP_PD6
- removed net 9: IC4.PCINT29/OC1A_PD5
- removed net A0: IC4.PCINT7/ADC7_PA7, JP9.1
- removed net A1: IC4.PCINT6/ADC6_PA6
- removed net A2: IC4.PCINT5/ADC5_PA5
- removed net A3: IC4.PCINT4/ADC4_PA4
- removed net A4: IC4.PCINT3/ADC3_PA3
- removed net A5: IC4.PCINT2/ADC2_PA2
- removed net A6: IC4.PCINT1/ADC1_PA1
- removed net A7: IC4.PCINT0/ADC0_PA0
- removed net AREF: C17.1, IC4.AREF
- removed net AVCC: C18.1, IC4.AVCC, L1.1
- removed net N$11: IC4.PCINT17/SDA_PC1, JP9.5
- removed net N$26: IC4.PCINT16/SCL_PC0, JP9.6
- removed net N$40: PI_PWR.2, PI_SW.1
- removed net N$5: C16.1, IC4.XTAL1, Y2.3
- removed net N$9: C11.1, IC4.XTAL2, Y2.1
- removed net PWM3: JP12.3
- removed net PWM4: JP13.3
- new net JP21: JP20.1, JP21.2
- new net MPU_INT: JP8.1
- new net N$48: C2.1, IC1.XTAL1, Y1.3
- new net N$49: C1.1, IC1.XTAL2, Y1.1
- new net PISUPPLY: C5.+, D1.C, IC3.IN, JP20.2
- new net SCL: IC1.(PCINT16/SCL)PC0, JP8.6
- new net SDA: IC1.(PCINT17/SDA)PC1, JP8.5
- new net TCK: IC1.(PCINT18/TCK)PC2, JTAG.1
- new net TDI: IC1.(PCINT21/TDI)PC5, JTAG.9
- new net TDO: IC1.(PCINT20/TDO)PC4, JTAG.3
- new net TMS: IC1.(PCINT19/TMS)PC3, JTAG.5
- new net US1ECHO: JP14.4, JP9.4
- new net US1TRIG: JP14.3, JP9.3
- new net VCC: IC1.VCC, IC1.VCC@1, IC1.VCC@2, JP6.10, JP6.9, JP7.10, JP7.9, JP8.8, JTAG.4
- net !RESET: now also IC1.RESET; no longer IC4.!RESET
- net 0(RX0): no longer IC4.PCINT24/RXD0_PD0
- net 1(TX0): no longer IC4.PCINT25/TXD0_PD1
- net 5V: now also C21.+, C8.1; no longer C19.1, C20.+, IC4.VCC, JP6.10, JP6.9, JP7.10, JP7.9, JP9.8, JTAG.4, L1.2
- net GND: now also C1.2, C2.2, C21.-, C8.2, IC1.GND, IC1.GND@1, IC1.GND@2, IC1.GND@3, JP14.1, JP21.1, JP8.7, JP9.1, Y1.2; no longer C11.2, C16.2, C17.2, C18.2, C19.2, C20.-, IC4.GND, IC4.GND@1, JP12.1, JP13.1, JP9.7, PI_PWR.1, Y2.2
- net VIN: now also JP14.2, JP9.2; no longer C5.+, D1.C, IC3.IN, JP12.2, JP13.2, PI_SW.2
Other:
- note added: "Resonator doesnt need caps, right?"
- note added: "This doesnt make sense. where is ground?"
- note added: "several 5V outputs, eg PI, LIDAR"
- note removed: "ATmega324/644/1284"
- note removed: "Do I need AREF or AVCC?"
- note removed: "Omit load capacitors if resonator"
- note removed: "USB Host for Pi Power"
- note removed: "fitted instead of crystal"
- moved on the sheet: JPX1, JPX10, JPX8, JTAG, U$1, U$4

Commit message: final mounting hole position on bd.
Parts:
- removed JP20: SW_1, pinhead:PINHD-1X2
- removed JP21: 5V_1, pinhead:PINHD-1X2
Connections:
- removed net JP21: JP20.1, JP21.2
- net GND: no longer JP21.1
- net PISUPPLY: no longer JP20.2
Other:
- note removed: "5V in from RC 5A switched regulator. Routed to Pi BUS via switch(or jumper). Also supplies Servos / Pings."
Changed lines of the file:
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@@
 <part name="JTAG" library="pinhead" deviceset="PINHD-2X5" device=""/>
 <part name="5V_IN" library="pinhead" deviceset="PINHD-1X2" device=""/>
-<part name="JP20" library="pinhead" deviceset="PINHD-1X2" device="" value="SW_1"/>
-<part name="JP21" library="pinhead" deviceset="PINHD-1X2" device="" value="5V_1"/>
 <part name="JPX1" library="pinhead" deviceset="PINHD-1X12" device=""/>
 <part name="U$1" library="s3-pilot2-lbr" deviceset="MC33926-SINGLE-BO" device="" value="M2"/>
@@
 11/7/2015 V3 started
 </text>
-<text x="276.86" y="109.22" size="1.778" layer="91">5V in from RC 5A switched regulator.
-Routed to Pi BUS via switch(or jumper).
-Also supplies Servos / Pings.</text>
 <text x="312.42" y="15.24" size="1.778" layer="97">3.3V
 150mA Out</text>
@@
 <instance part="JTAG" gate="A" x="601.98" y="111.76"/>
 <instance part="5V_IN" gate="G$1" x="264.16" y="93.98" rot="R180"/>
-<instance part="JP20" gate="G$1" x="264.16" y="137.16" rot="R180"/>
-<instance part="JP21" gate="G$1" x="264.16" y="121.92" rot="R180"/>
 <instance part="JPX1" gate="G$1" x="563.88" y="-2.54"/>
 <instance part="U$1" gate="G$1" x="525.78" y="-2.54" rot="R180"/>
@@
 </segment>
 <segment>
-<pinref part="JP21" gate="G$1" pin="1"/>
-<wire x1="266.7" y1="119.38" x2="276.86" y2="119.38" width="0.1524" layer="91"/>
-<label x="279.4" y="119.38" size="1.778" layer="95"/>
-</segment>
-<segment>
 <pinref part="C1" gate="G$1" pin="2"/>
 <pinref part="GND3" gate="1" pin="GND"/>
@@
 </segment>
 </net>
-<net name="JP21" class="0">
-<segment>
-<pinref part="JP20" gate="G$1" pin="1"/>
-<wire x1="266.7" y1="134.62" x2="276.86" y2="134.62" width="0.1524" layer="91"/>
-<pinref part="JP21" gate="G$1" pin="2"/>
-<wire x1="266.7" y1="121.92" x2="276.86" y2="121.92" width="0.1524" layer="91"/>
-<wire x1="276.86" y1="134.62" x2="276.86" y2="121.92" width="0.1524" layer="91"/>
-</segment>
-</net>
 <net name="N$18" class="0">
 <segment>
@@
 <net name="PISUPPLY" class="0">
 <segment>
-<pinref part="JP20" gate="G$1" pin="2"/>
-<wire x1="276.86" y1="137.16" x2="266.7" y2="137.16" width="0.1524" layer="91"/>
-<label x="276.86" y="137.16" size="1.778" layer="95"/>
-</segment>
-<segment>
 <wire x1="299.72" y1="93.98" x2="297.18" y2="93.98" width="0.1524" layer="91"/>

Commit message: .
Parts:
- C1, C2, C8: device SparkFun:CAPPTH -> SparkFun:CAP0603-CAP
- C21: device SparkFun:CAP_POLPTH2 -> SparkFun:CAP_POL1206
- JP2: value ESC_ENA -> ENA
Changed lines of the file:
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@@
 <grid distance="0.1" unitdist="inch" unit="inch" style="lines" multiple="1" display="no" altdistance="0.01" altunitdist="inch" altunit="inch"/>
 <layers>
-<layer number="1" name="Top" color="4" fill="1" visible="no" active="no"/>
-<layer number="2" name="Route2" color="1" fill="3" visible="no" active="no"/>
-<layer number="3" name="Route3" color="4" fill="3" visible="no" active="no"/>
-<layer number="14" name="Route14" color="1" fill="6" visible="no" active="no"/>
-<layer number="15" name="Route15" color="4" fill="6" visible="no" active="no"/>
-<layer number="16" name="Bottom" color="1" fill="1" visible="no" active="no"/>
-<layer number="17" name="Pads" color="2" fill="1" visible="no" active="no"/>
-<layer number="18" name="Vias" color="2" fill="1" visible="no" active="no"/>
-<layer number="19" name="Unrouted" color="6" fill="1" visible="no" active="no"/>
-<layer number="20" name="Dimension" color="15" fill="1" visible="no" active="no"/>
-<layer number="21" name="tPlace" color="7" fill="1" visible="no" active="no"/>
-<layer number="22" name="bPlace" color="7" fill="1" visible="no" active="no"/>
-<layer number="23" name="tOrigins" color="15" fill="1" visible="no" active="no"/>
-<layer number="24" name="bOrigins" color="15" fill="1" visible="no" active="no"/>
-<layer number="25" name="tNames" color="7" fill="1" visible="no" active="no"/>
-<layer number="26" name="bNames" color="7" fill="1" visible="no" active="no"/>
-<layer number="27" name="tValues" color="7" fill="1" visible="no" active="no"/>
-<layer number="28" name="bValues" color="7" fill="1" visible="no" active="no"/>
+<layer number="1" name="Top" color="4" fill="1" visible="yes" active="no"/>
+<layer number="2" name="Route2" color="1" fill="3" visible="yes" active="no"/>
+<layer number="3" name="Route3" color="4" fill="3" visible="yes" active="no"/>
+<layer number="14" name="Route14" color="1" fill="6" visible="yes" active="no"/>
+<layer number="15" name="Route15" color="4" fill="6" visible="yes" active="no"/>
+<layer number="16" name="Bottom" color="1" fill="1" visible="yes" active="no"/>
+<layer number="17" name="Pads" color="2" fill="1" visible="yes" active="no"/>
+<layer number="18" name="Vias" color="2" fill="1" visible="yes" active="no"/>
+<layer number="19" name="Unrouted" color="6" fill="1" visible="yes" active="no"/>
+<layer number="20" name="Dimension" color="15" fill="1" visible="yes" active="no"/>
+<layer number="21" name="tPlace" color="7" fill="1" visible="yes" active="no"/>
+<layer number="22" name="bPlace" color="7" fill="1" visible="yes" active="no"/>
+<layer number="23" name="tOrigins" color="15" fill="1" visible="yes" active="no"/>
+<layer number="24" name="bOrigins" color="15" fill="1" visible="yes" active="no"/>
+<layer number="25" name="tNames" color="7" fill="1" visible="yes" active="no"/>
+<layer number="26" name="bNames" color="7" fill="1" visible="yes" active="no"/>
+<layer number="27" name="tValues" color="7" fill="1" visible="yes" active="no"/>
+<layer number="28" name="bValues" color="7" fill="1" visible="yes" active="no"/>
 <layer number="29" name="tStop" color="7" fill="3" visible="no" active="no"/>
 <layer number="30" name="bStop" color="7" fill="6" visible="no" active="no"/>
@@
 <layer number="35" name="tGlue" color="7" fill="4" visible="no" active="no"/>
 <layer number="36" name="bGlue" color="7" fill="5" visible="no" active="no"/>
-<layer number="37" name="tTest" color="7" fill="1" visible="no" active="no"/>
-<layer number="38" name="bTest" color="7" fill="1" visible="no" active="no"/>
+<layer number="37" name="tTest" color="7" fill="1" visible="yes" active="no"/>
+<layer number="38" name="bTest" color="7" fill="1" visible="yes" active="no"/>
 <layer number="39" name="tKeepout" color="4" fill="11" visible="no" active="no"/>
 <layer number="40" name="bKeepout" color="1" fill="11" visible="no" active="no"/>
@@
 <layer number="44" name="Drills" color="7" fill="1" visible="no" active="no"/>
 <layer number="45" name="Holes" color="7" fill="1" visible="no" active="no"/>
-<layer number="46" name="Milling" color="3" fill="1" visible="no" active="no"/>
-<layer number="47" name="Measures" color="7" fill="1" visible="no" active="no"/>
-<layer number="48" name="Document" color="7" fill="1" visible="no" active="no"/>
-<layer number="49" name="Reference" color="7" fill="1" visible="no" active="no"/>
-<layer number="50" name="dxf" color="7" fill="1" visible="no" active="no"/>
-<layer number="51" name="tDocu" color="7" fill="1" visible="no" active="no"/>
-<layer number="52" name="bDocu" color="7" fill="1" visible="no" active="no"/>
-<layer number="53" name="tGND_GNDA" color="7" fill="9" visible="no" active="no"/>
-<layer number="54" name="bGND_GNDA" color="1" fill="9" visible="no" active="no"/>
-<layer number="56" name="wert" color="7" fill="1" visible="no" active="no"/>
-<layer number="57" name="tCAD" color="7" fill="1" visible="no" active="no"/>
+<layer number="46" name="Milling" color="3" fill="1" visible="yes" active="no"/>
+<layer number="47" name="Measures" color="7" fill="1" visible="yes" active="no"/>
+<layer number="48" name="Document" color="7" fill="1" visible="yes" active="no"/>
+<layer number="49" name="Reference" color="7" fill="1" visible="yes" active="no"/>
+<layer number="50" name="dxf" color="7" fill="1" visible="yes" active="no"/>
+<layer number="51" name="tDocu" color="7" fill="1" visible="yes" active="no"/>
+<layer number="52" name="bDocu" color="7" fill="1" visible="yes" active="no"/>
+<layer number="53" name="tGND_GNDA" color="7" fill="9" visible="yes" active="no"/>
+<layer number="54" name="bGND_GNDA" color="1" fill="9" visible="yes" active="no"/>
+<layer number="56" name="wert" color="7" fill="1" visible="yes" active="no"/>
+<layer number="57" name="tCAD" color="7" fill="1" visible="yes" active="no"/>
 <layer number="90" name="Modules" color="5" fill="1" visible="no" active="yes"/>
 <layer number="91" name="Nets" color="2" fill="1" visible="yes" active="yes"/>
@@
 <parts>
 <part name="MPU6050" library="s3-pilot2-lbr" deviceset="MPU-6050-BO" device=""/>
-<part name="JP2" library="pinhead" deviceset="PINHD-1X2" device="" value="ESC_ENA"/>
+<part name="JP2" library="pinhead" deviceset="PINHD-1X2" device="" value="ENA"/>
 <part name="GND1" library="SparkFun-Aesthetics" deviceset="GND" device=""/>
 <part name="JP10" library="pinhead" deviceset="PINHD-1X3" device="/90" value="PWM1"/>
@@
 <part name="U$1" library="s3-pilot2-lbr" deviceset="MC33926-SINGLE-BO" device="" value="M2"/>
 <part name="IC1" library="atmel" deviceset="ATMEGA644" device="A"/>
-<part name="C1" library="SparkFun" deviceset="CAP" device="PTH" value="22p">
+<part name="C1" library="SparkFun" deviceset="CAP" device="0603-CAP" value="22p">
 <attribute name="OPTION" value="Do not fit for ceramic resonator"/>
 </part>
-<part name="C2" library="SparkFun" deviceset="CAP" device="PTH" value="22p">
+<part name="C2" library="SparkFun" deviceset="CAP" device="0603-CAP" value="22p">
 <attribute name="OPTION" value="Do not fit for ceramic resonator"/>
 </part>
@@
 <part name="GND4" library="supply1" deviceset="GND" device=""/>
 <part name="5V1" library="supply1" deviceset="VCC" device=""/>
-<part name="C8" library="SparkFun" deviceset="CAP" device="PTH" value="100n"/>
-<part name="C21" library="SparkFun" deviceset="CAP_POL" device="PTH2" value="4u7"/>
+<part name="C8" library="SparkFun" deviceset="CAP" device="0603-CAP" value="100n"/>
+<part name="C21" library="SparkFun" deviceset="CAP_POL" device="1206" value="4u7"/>
 <part name="Y1" library="SteveMarple" deviceset="CRYSTAL-RESONATOR" device="" value="16MHz">
 <attribute name="OPTION" value="Crystal or ceramic resonator. Max 12MHz for 3V3 operation."/>

Commit message: .
Parts:
- removed 5V_IN: (no value), pinhead:PINHD-1X2
- removed C2: 22p, SparkFun:CAP0603-CAP
- removed JP1: Reset, pinhead:PINHD-1X2
- added JP12: PWM3, pinhead:PINHD-1X3/90
- added X1, X2: 5V, con-phoenix-350:1751248
- C1: value 22p -> 47pF; device SparkFun:CAP0603-CAP -> SparkFun-Capacitors:47PF-50V-5%(0603); OPTION Do not fit for ceramic resonator -> (none)
Connections:
- net 0(RX0) renamed RX
- net 1(TX0) renamed TX
- removed net N$24: 5V_IN.1, Q1.G, R5.1
- removed net N$36: 5V_IN.2, D1.A
- removed net VCC: IC1.VCC, IC1.VCC@1, IC1.VCC@2, JP6.10, JP6.9, JP7.10, JP7.9, JP8.8, JTAG.4
- removed net VIN: JP10.2, JP11.2, JP14.2, JP9.2
- new net N$11: C1.1, U2.BP
- new net N$5: Q1.G, R5.1
- new net N$9: D1.A, X1-2.K, X2-2.K
- new net PWM3: JP12.3
- net !RESET: no longer JP1.2
- net 5V: now also IC1.VCC, IC1.VCC@1, IC1.VCC@2, JP10.2, JP11.2, JP12.2, JP14.2, JP6.10, JP6.9, JP7.10, JP7.9, JP8.8, JP9.2, JTAG.4
- net GND: now also JP12.1, X1-1.K, X2-1.K; no longer C2.2, JP1.1
- net N$48: no longer C2.1
- net N$49: no longer C1.1
Other:
- note added: "need to finish this with a switch usb vs 5v in supplying 3.3v regulator"
- note removed: "Resonator doesnt need caps, right?"
- note removed: "This doesnt make sense. where is ground?"
- note removed: "several 5V outputs, eg PI, LIDAR"
- moved on the sheet: C1, C21, C3, C4, C5, C6, C7, C8, D1, IC1, IC3, JP10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
