File: s3-pilot3.sch (EAGLE design)
At the start: 65 parts, among them IC1 ATMEGA644A, IC3 LM1117, Q1 ZXMP6A13FTA, Q2 2N7002PW, U1 FT231XS, U2 MIC5205, X1 5V, X2 5V, Y1 16MHz

Commit message: .
Parts:
- removed IC1: ATMEGA644A, atmel:ATMEGA644A
- removed JTAG: (no value), pinhead:PINHD-2X5
- removed Y1: 16MHz, SteveMarple:CRYSTAL-RESONATOR
- added IC2: XMEGA16A4A, atmel:XMEGA16A4A
- added JP1: (no value), pinhead:PINHD-1X3
- added U$2: JTAG, s3-pilot2-lbr:CON-JTAG
- added Y2: 16MHz, SteveMarple:CRYSTAL-RESONATOR
- JP8: value MPU-6050 -> IMU
Connections:
- removed net N$48: IC1.XTAL1, Y1.3
- removed net N$49: IC1.XTAL2, Y1.1
- new net N$24: JP1.2, Q1.G
- new net N$26: JPX10.8, MPU6050.INT
- new net N$36: IC2.PR0(XT2), Y2.3
- new net N$40: IC2.PR1(XT1), Y2.1
- net !RESET: now also IC2.!RESET!/PDI_CLK, U$2.!RESET; no longer IC1.RESET, JTAG.6
- net 5V: now also IC2.VCC, IC2.VCC1, IC2.VCC2, U$2.VCC; no longer IC1.VCC, IC1.VCC@1, IC1.VCC@2, JPX10.8, JTAG.4, MPU6050.VCC
- net GND: now also IC2.GND, IC2.GND1, IC2.GND2, IC2.GND3, JP1.3, U$2.GND, U$2.GND@1, Y2.2; no longer IC1.GND, IC1.GND@1, IC1.GND@2, IC1.GND@3, JTAG.10, JTAG.2, Y1.2
- net N$13: now also MPU6050.VCC; no longer MPU6050.INT
- net N$14: now also MPU6050.GND; no longer MPU6050.AD0
- net N$16: now also MPU6050.SCL; no longer MPU6050.XCL
- net N$17: now also MPU6050.SDA; no longer MPU6050.XDA
- net N$19: now also MPU6050.XDA; no longer MPU6050.SDA
- net N$20: now also MPU6050.XCL; no longer MPU6050.SCL
- net N$22: now also MPU6050.AD0; no longer MPU6050.GND
- net N$5: now also JP1.1; no longer Q1.G
- net RX: now also IC2.PD0
- net SCL: now also IC2.PC0; no longer IC1.(PCINT16/SCL)PC0
- net SDA: now also IC2.PC1; no longer IC1.(PCINT17/SDA)PC1
- net TCK: now also IC2.PC2, U$2.TCK; no longer IC1.(PCINT18/TCK)PC2, JTAG.1
- net TDI: now also IC2.PC5, U$2.TDI; no longer IC1.(PCINT21/TDI)PC5, JTAG.9
- net TDO: now also IC2.PC4, U$2.TDO; no longer IC1.(PCINT20/TDO)PC4, JTAG.3
- net TMS: now also IC2.PC3, U$2.TMS; no longer IC1.(PCINT19/TMS)PC3, JTAG.5
- net TX: now also IC2.PD1
Other:
- note added: "need to finish DTR"
- moved on the sheet: C1, C10, C12, C13, C14, C15, C21, C3, C4, C5, C6, C7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
