File: s3-pilot3.sch (EAGLE design)
At the start: 66 parts, among them IC2 XMEGA16A4A, IC3 LM1117, Q1 ZXMP6A13FTA, Q2 2N7002PW, U1 FT231XS, U2 MIC5205, X1 5V, X2 5V, Y2 16MHz

Commit message: .
Parts:
- added C2: 0.1uF, SparkFun:CAP0805
- added R4: 10k, SparkFun:RESISTOR0603-RES
Connections:
- removed net N$5: JP1.1, R5.1
- removed net N$9: D1.A, X1-2.K, X2-2.K
- new net 5VIN: D1.A, JP1.1, JP10.2, JP11.2, JP12.2, R5.1, X1-2.K, X2-2.K
- net !RESET: now also C2.2, R4.1
- net 3.3V: now also JP8.8
- net 5V: now also R4.2; no longer JP10.2, JP11.2, JP12.2, JP8.8
- net DTR: now also C2.1
Other:
- note removed: "need to finish DTR"
- note removed: "need to finish this with a switch usb vs 5v in supplying 3.3v regulator"
- moved on the sheet: C1, C12, C3, C4, C5, C6, C7, D1, IC3, JP1, JP5, LED1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

Commit message: .
Parts:
- JP1: value (none) -> 3V-5V
- Y2: value 16MHz -> 16Mhz; device SteveMarple:CRYSTAL-RESONATOR -> s3-pilot2-lbr:SMD-RESONATOR-KYOCERA-PBRV-H
Other:
- moved on the sheet: C12, C14, C15, C2, IC2, JPX10, R4, Y2
