File: s3-pilot3.brd (EAGLE design)
At the start: 85 x 56 mm, 74 parts, among them IC2 XMEGA16A4A, IC3 LM1117, Q1 ZXMP6A13FTA, Q2 2N7002PW, U1 FT231XS, U2 MIC5205, X1 5V, X2 5V, Y2 16MHz

Commit message: .
Parts:
- added C2: 0.1uF, SparkFun:0805
- added E$1, E$4: (no value), holes:2,8
- added R4: 10k, SparkFun:0603-RES
- moved R14 59.3 mm to (71.1, 2.54), turned to 180 degrees
- moved R15 58.6 mm to (67.3, 2.54)
- moved JP1 43.3 mm to (44.5, 7.62)
- moved C15 34.2 mm to (71.1, 26.7)
- moved LED3 33.0 mm to (82.5, 52.1), turned to 90 degrees
- moved C6 31.2 mm to (71.1, 20.3), turned to 90 degrees
- moved C3 30.2 mm to (71.1, 14.0), turned to 90 degrees
- moved C4 30.2 mm to (66.0, 16.5), turned to 0 degrees
- moved R7 29.9 mm to (82.5, 47.0), turned to 90 degrees
- moved R5 29.7 mm to (55.9, 17.8), turned to 90 degrees
- moved JP2 27.7 mm to (68.6, 52.1), turned to 0 degrees
- moved LED4 26.7 mm to (82.5, 41.9), turned to 90 degrees
- moved JP5 25.4 mm to (44.5, 53.3)
- moved C12 25.0 mm to (81.3, 21.6), turned to 0 degrees
- moved R9 23.1 mm to (82.7, 36.8), turned to 90 degrees
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Connections:
- removed net N$5: JP1.1, R5.1
- removed net N$9: D1.A, X1.2, X2.2
- new net 5VIN: D1.A, JP1.1, JP10.2, JP11.2, JP12.2, R5.1, X1.2, X2.2
- net !RESET: now also C2.2, R4.1
- net 3.3V: now also JP8.8
- net 5V: now also R4.2; no longer JP10.2, JP11.2, JP12.2, JP8.8
- net DTR: now also C2.1
Routing:
- net GND: track 0.00 -> 464.8 mm, vias 0 -> 4
- net 5V: track 0.00 -> 370.7 mm, vias 0 -> 8
- net 5VIN: track 0.00 -> 160.3 mm
- net ESC_ENA: track 0.00 -> 147.8 mm, vias 0 -> 1
- net RX: track 0.00 -> 107.5 mm, vias 0 -> 4
- net !RESET: track 0.00 -> 96.0 mm, vias 0 -> 5
- net 3.3V: track 0.00 -> 95.2 mm, vias 0 -> 6
- net RXLED: track 0.00 -> 72.4 mm, vias 0 -> 4
- net USBVCC: track 0.00 -> 60.6 mm, vias 0 -> 4
- net TXLED: track 0.00 -> 54.0 mm, vias 0 -> 2
- net TX: track 0.00 -> 46.4 mm, vias 0 -> 2
- net SDA: track 0.00 -> 44.0 mm, vias 0 -> 1
- net D+: track 0.00 -> 40.4 mm, vias 0 -> 2
- net SCL: track 0.00 -> 40.1 mm, vias 0 -> 1
- net US1TRIG: track 0.00 -> 28.1 mm
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
Commit message: .
Parts:
- JP1: value (none) -> 3V-5V
- Y2: value 16MHz -> 16Mhz; device SteveMarple:HC49U-V-RESONATOR -> s3-pilot2-lbr:SMD-KYOCERA-PBRV-H
- moved U$1 38.7 mm to (88.9, 87.6)
- moved JPX1 37.4 mm to (96.5, 78.7)
- moved JP2 26.9 mm to (43.2, 43.2)
- moved JPX10 26.1 mm to (58.4, 77.5)
- moved MPU6050 21.8 mm to (68.6, 82.5)
- moved Y2 5.08 mm to (50.8, 43.2), turned to 90 degrees
- moved JPX8 3.81 mm to (24.1, 94.0)
- moved C8 1.42 mm to (57.1, 47.6), turned to 270 degrees
- moved IC3 1.27 mm to (69.6, 7.35)
- moved U1 0.90 mm to (64.1, 25.4)
Connections:
- net GND: now also Y2.2; no longer Y2.GND
- net N$36: now also Y2.3; no longer Y2.2
Routing:
- net RX: track 107.5 -> 15.6 mm, vias 4 -> 2
- net 5V: track 370.7 -> 306.0 mm, vias 8 -> 4
- net D-: track 20.0 -> 77.2 mm
- net GND: track 464.8 -> 421.3 mm, vias 4 -> 8
- net DTR: track 26.7 -> 67.3 mm, vias 3 -> 4
- net ESC_ENA: track 147.8 -> 107.6 mm
- net TX: track 46.4 -> 13.7 mm
- net !RESET: track 96.0 -> 65.2 mm
- net D+: track 40.4 -> 66.0 mm, vias 2 -> 3
- net 3.3V: track 95.2 -> 119.6 mm, vias 6 -> 4
- net SDA: track 44.0 -> 62.3 mm
- net RXLED: track 72.4 -> 57.2 mm, vias 4 -> 2
- net 5VIN: track 160.3 -> 148.1 mm, vias 0 -> 1
- net N$36: track 19.4 -> 8.36 mm, vias 1 -> 0
- net TMS: track 16.3 -> 25.2 mm
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- added copper zone on layer 1, net GND
- added copper zone on layer 16, net GND
